File: astable-ttl.sch (KiCad schematic (older format))
At the start: 9 parts

Commit message: modified the automatic circuit
Parts:
- removed C? (x2): C, symbol C
- removed J? (x2): Conn_01x02, symbol Conn_01x02
- removed J?: Conn_01x01, symbol Conn_01x01
- removed R?: R, symbol R
- removed RV? (x2): POT, symbol POT
- added C1: 0.1UF, Capacitors_THT:C_Disc_D3.8mm_W2.6mm_P2.50mm, symbol C
- added C2, C4: 100UF, Capacitors_THT:CP_Radial_D8.0mm_P2.50mm, symbol C
- added C3: 10UF, Capacitors_THT:CP_Radial_D5.0mm_P2.00mm, symbol C
- added D1: LED, LEDs:LED_D3.0mm, symbol LED
- added R1: 330, Resistors_THT:R_Axial_DIN0207_L6.3mm_D2.5mm_P7.62mm_Horizontal, symbol R
- added R2: 5K, Resistors_THT:R_Axial_DIN0207_L6.3mm_D2.5mm_P7.62mm_Horizontal, symbol R
- added RV1: POT, Potentiometers:Potentiometer_Triwood_RM-065, symbol POT
- added U2: L7805, TO_SOT_Packages_THT:TO-220_Vertical, symbol L7805
- added U3: Barrel_jack, library:Barrel_jack, symbol Barrel_jack
- U1: renamed from U?; footprint (none) -> Housings_DIP:DIP-8_W7.62mm
Connections:
- net labels removed: OUT, SIG
- wire segments 7 -> 32
- no-connect marks 0 -> 1
Other:
- moved on the sheet: U1
