File: Automatic3.0/Power_Supply.sch (KiCad schematic (older format))
At the start: 31 parts, among them J16 CONN_01X02, J17 Reset_Jumper, J18 Reset_Jumper, SW1 Reset, SW2 Reset, U3 Buck, U4 LM7809

Commit message: modified the automatic circuit
Parts:
- removed D12: LED_5V, modFiles:LED_D3.0mm, symbol LED
- removed R19: 330, modFiles:Resistor_small, symbol R
- added C13: 100uF, modFiles:Capacitor_100uF, symbol C
- added C4: 1000uF, modFiles:Capacitor_1000uF, symbol C
- added D12: D, Diodes_THT:D_DO-27_P12.70mm_Horizontal, symbol D
- added D17, D20: LED, modFiles:LED_D3.0mm, symbol LED
- added D19: LED_5V, modFiles:LED_D3.0mm, symbol LED
- added F3: Fuse, modFiles:Fuse_Holder, symbol Fuse
- added J22, J23: CONN_01X02, modFiles:Connector_Bornier_2, symbol CONN_01X02
- added R35, R42, R43: 330, modFiles:Resistor_small, symbol R
- added U5: Buck, modFiles:Buck_Regulator, symbol Buck
- U3: value Buck -> Buck_5A
Connections:
- net +12V: now also F3.2
- net +5V: now also C13.1, U5.3 (OUT(+)); no longer C11.1, U3.3 (OUT(+))
- net 5V: no longer J17.1 (P1)
- net BUCK: now also C4.1, U5.1 (IN(+)); no longer C8.1, U3.1 (IN(+))
- net GND: now also C13.2, C4.2, D17.1 (K), D19.1 (K), D20.1 (K), J22.2 (P2), J23.1 (P1), U5.2 (IN(-)), U5.4 (OUT(-))
- net at C9.1, D10.1 (K), U4.1 (IN): now also R42.2
- new net: C11.1, J22.1 (P1), J23.2 (P2), R43.2, U3.3 (OUT(+))
- new net: D19.2 (A), R35.1
- new net: D12.2 (A), F3.1
- new net: D20.2 (A), R43.1
- new net: D17.2 (A), R42.1
- new net 12V: C8.1, D12.1 (K), U3.1 (IN(+))
- new net 3V3: J17.1 (P1), R35.2
Other:
- moved on the sheet: C11, C8, J17, J18, R21, R22, SW1, SW2, U3
