File: Automatic3.0/Automatic3.kicad_pcb (KiCad board)
At the start: 2 copper layers, 87 parts, among them J1 GND VCC, J10 Line Tracker and Proximity, J11 Compass, J12 Bluetooth, J13 Encoder, J14 Bluetooth, J15 Motor, J16 CONN_01X02, J17 Reset_Jumper, J18 Reset_Jumper, J19 Bluetooth, J2 CONN_01X01, J4 CONN_01X01, J5 CONN_01X01, J6 I/O Pins, J7 USB_B, J8 CONN_01X01, J9 I/O Pins, SW1 Reset, SW2 Reset, U1 Arduino_Mega2560_Shield, U2 Arduino_Mega2560_Shield, U3 Buck, U4 LM7809

Commit message: modified the automatic circuit
Parts:
- removed C12: 104, modFiles:Capacitor_Disc_Medium
- removed D15: D_Zener, Diodes_THT:D_DO-35_SOD27_P7.62mm_Horizontal
- removed D16: LED, modFiles:LED_D3.0mm
- removed R19: 330, modFiles:Resistor_small
- removed R29, R30: R, modFiles:Resistor_small
- added C13: 100uF, modFiles:Capacitor_100uF, F.Cu at (76.7, 114.0)
- added C4: 1000uF, modFiles:Capacitor_1000uF, F.Cu at (86.8, 62.1)
- added D18: D_Zener, Diodes_THT:D_DO-35_SOD27_P7.62mm_Horizontal, F.Cu at (230.4, 108.6)
- added D19: LED_5V, modFiles:LED_D3.0mm, F.Cu at (135.2, 73.0)
- added D20: LED, modFiles:LED_D3.0mm, F.Cu at (47.7, -11.9)
- added F3: Fuse, modFiles:Fuse_Holder, F.Cu at (167.4, 80.9)
- added J20: Bluetooth, Pin_Headers:Pin_Header_Straight_1x06_Pitch2.54mm, F.Cu at (94.9, 108.0)
- added J21: CONN_01X02, modFiles:Connector_Bornier_2, F.Cu at (151.0, 44.0)
- added J22: CONN_01X02, modFiles:Connector_Bornier_2, F.Cu at (167.1, 128.1)
- added J23: CONN_01X02, modFiles:Connector_Bornier_2, F.Cu at (167.3, 117.9)
- added Q2: IRF540N, modFiles:Voltage_Regulators, F.Cu at (199.0, -7.26)
- added Q3: IRF540N, modFiles:Voltage_Regulators, F.Cu at (199.2, -17.4)
- added R31: R, modFiles:Resistor_small, F.Cu at (95.5, 55.8)
- added R32: R, modFiles:Resistor_small, F.Cu at (221.4, 131.1)
- added R33: R, modFiles:Resistor_small, F.Cu at (125.4, 121.4)
- added R34: R, modFiles:Resistor_small, F.Cu at (125.3, 118.0)
- added R35: 330, modFiles:Resistor_small, F.Cu at (138.3, 69.1)
- added R36: 560, modFiles:Resistor_small, F.Cu at (227.3, 2.25)
- added R37: 560, modFiles:Resistor_small, F.Cu at (224.1, -9.66)
- added R38: 10k, modFiles:Resistor_small, F.Cu at (231.0, -3.26)
- added R39: 10k, modFiles:Resistor_small, F.Cu at (212.4, -19.2)
- added R42: 330, modFiles:Resistor_small, F.Cu at (67.9, 69.6)
- added R43: 330, modFiles:Resistor_small, F.Cu at (56.3, -3.04)
- added U5: Buck, modFiles:Buck_Regulator, F.Cu at (89.5, 70.0)
- D12: value LED_5V -> D; footprint modFiles:LED_D3.0mm -> Diodes_THT:D_DO-27_P12.70mm_Horizontal
- D2, D3: footprint modFiles:Diode_Small -> modFiles:Diode_small
- D4: value D_Zener -> LED; footprint Diodes_THT:D_DO-35_SOD27_P7.62mm_Horizontal -> modFiles:LED_D3.0mm
- J11: footprint Connectors_JST:JST_PH_B4B-PH-K_04x2.00mm_Straight -> Connectors_JST:JST_XH_B04B-XH-A_04x2.50mm_Straight
- J19: value Bluetooth -> CONN_01X02; footprint Pin_Headers:Pin_Header_Straight_1x06_Pitch2.54mm -> modFiles:Connector_Bornier_2
- J2, J4, J5, J8: footprint Connectors:1pin -> modFiles:1_Pin
- J6: value I/O Pins -> Zone_Switches; footprint Pin_Headers:Pin_Header_Straight_1x08_Pitch2.54mm -> modFiles:Connector_DB_9
- J7: value USB_B -> Throwing; footprint Connectors_JST:JST_PH_B4B-PH-K_04x2.00mm_Straight -> Connectors_JST:JST_XH_B04B-XH-A_04x2.50mm_Straight
- U3: value Buck -> Buck_5A
- moved C11 140.9 mm to (211.5, 82.4), turned to 270 degrees
- moved C8 126.3 mm to (215.1, 44.4)
- moved D17 99.2 mm to (67.5, 75.5), turned to 90 degrees
- moved J19 91.9 mm to (161.3, 44.0)
- moved J2 82.5 mm to (249.5, 120.9)
- moved D4 76.3 mm to (90.8, 52.7), turned to 0 degrees
- moved C6 63.7 mm to (200.4, 42.7)
- moved R25 63.3 mm to (20.8, 94.9)
- moved R27 62.9 mm to (184.3, 100.8)
- moved R26 61.7 mm to (22.8, 105.8)
- moved J6 55.8 mm to (100.2, 46.9), turned to 0 degrees
- moved J4 54.9 mm to (218.9, 20.7)
- moved F2 47.3 mm to (168.4, 53.0), turned to 90 degrees
- moved U3 46.3 mm to (116.0, 103.0), turned to 0 degrees
- moved D9 37.6 mm to (67.1, 94.6), turned to 90 degrees
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Connections:
- net Net-(J6-Pad8) renamed /PF0
- C11 pad 1: +5V -> Net-(C11-Pad1)
- C6 pad 1: +5V -> /3V3
- C8 pad 1: /12VV -> /12Vin
- D1 pad 1: /TX2 -> /TX3
- D12 pad 1: GND -> /12Vin
- D4 pad 1: /TX0 -> GND
- D4 pad 2: GND -> Net-(D4-Pad2)
- J11 pad 1: +5V -> /3V3
- J12 pad 1: Net-(J12-Pad1) -> (no net)
- J12 pad 4: /RX2 -> /RX3
- J12 pad 5: /TX2 -> /TX3
- J12 pad 6: Net-(J12-Pad6) -> (no net)
- J14 pad 1: Net-(J14-Pad1) -> (no net)
- J14 pad 6: Net-(J14-Pad6) -> (no net)
- J17 pad 1: /5VV -> /3V3
- J19 pad 1: Net-(J19-Pad1) -> /12Vin
- J19 pad 2: +5V -> Net-(J19-Pad2)
- J6 pad 1: Net-(J6-Pad1) -> /PF6
- J6 pad 2: Net-(J6-Pad2) -> /PF5
- J6 pad 3: Net-(J6-Pad3) -> /PF4
- J6 pad 4: Net-(J6-Pad4) -> /PF3
- J6 pad 5: Net-(J6-Pad5) -> /PF2
- J6 pad 6: Net-(J6-Pad6) -> GND
- J6 pad 7: Net-(J6-Pad7) -> (no net)
- R23 pad 1: +5V -> /3V3
- R24 pad 1: +5V -> /3V3
- U1 pad 11: Net-(R30-Pad2) -> (no net)
- U1 pad 12: Net-(R29-Pad2) -> (no net)
- U1 pad 2: Net-(U1-Pad2) -> (no net)
- U1 pad 23: Net-(U1-Pad23) -> (no net)
- U1 pad 24: Net-(U1-Pad24) -> (no net)
- U1 pad 25: Net-(U1-Pad25) -> (no net)
- U1 pad 3V3: Net-(U1-Pad3V3) -> /3V3
- U1 pad 4: Net-(U1-Pad4) -> (no net)
- U1 pad 42: Net-(U1-Pad42) -> (no net)
- U1 pad 44: Net-(U1-Pad44) -> (no net)
- U1 pad 46: Net-(U1-Pad46) -> (no net)
- U1 pad 47: Net-(U1-Pad47) -> (no net)
- U1 pad 5: Net-(U1-Pad5) -> (no net)
- U1 pad 5V1: /5VV -> (no net)
- U1 pad 6: Net-(U1-Pad6) -> (no net)
- U1 pad 8: Net-(U1-Pad8) -> (no net)
- U1 pad 9: Net-(U1-Pad9) -> (no net)
- U1 pad A1: Net-(J6-Pad7) -> /PF1
- U1 pad A12: Net-(U1-PadA12) -> (no net)
- U1 pad A13: Net-(U1-PadA13) -> (no net)
- U1 pad A14: Net-(U1-PadA14) -> (no net)
- U1 pad A2: Net-(J6-Pad6) -> /PF2
- U1 pad A3: Net-(J6-Pad5) -> /PF3
- U1 pad A4: Net-(J6-Pad4) -> /PF4
- U1 pad A5: Net-(J6-Pad3) -> /PF5
- U1 pad A6: Net-(J6-Pad2) -> /PF6
- U1 pad A7: Net-(J6-Pad1) -> (no net)
- U1 pad AREF: Net-(U1-PadAREF) -> (no net)
- U2 pad 0: Net-(U2-Pad0) -> (no net)
- U2 pad 1: Net-(U2-Pad1) -> (no net)
- U2 pad 11: Net-(U2-Pad11) -> (no net)
- U2 pad 22: Net-(U2-Pad22) -> (no net)
- U2 pad 27: Net-(U2-Pad27) -> (no net)
- U2 pad 28: Net-(U2-Pad28) -> (no net)
- U2 pad 29: Net-(U2-Pad29) -> (no net)
- U2 pad 30: Net-(U2-Pad30) -> (no net)
- U2 pad 31: Net-(U2-Pad31) -> (no net)
- U2 pad 32: Net-(U2-Pad32) -> (no net)
- U2 pad 33: Net-(U2-Pad33) -> (no net)
- U2 pad 3V3: Net-(U2-Pad3V3) -> (no net)
- U2 pad 47: Net-(U2-Pad47) -> (no net)
- U2 pad 8: Net-(U2-Pad8) -> (no net)
- U2 pad 9: Net-(U2-Pad9) -> (no net)
- U2 pad AREF: Net-(U2-PadAREF) -> (no net)
- U2 pad SCL: /SCL -> (no net)
- U2 pad SDA: /SDA -> (no net)
- U3 pad 1: /12VV -> /12Vin
- U3 pad 3: +5V -> Net-(C11-Pad1)
Routing:
- net +5V: track 425.2 -> 120.2 mm, vias 4 -> 0
- net GND: track 281.6 -> 65.5 mm
- net /TX2: track 107.9 -> 0.00 mm, vias 2 -> 0
- net /SDA: track 107.5 -> 0.00 mm, vias 2 -> 0
- net /INT5: track 113.3 -> 14.8 mm, vias 2 -> 0
- net Net-(D11-Pad2): track 6.41 -> 102.7 mm
- net /SCL: track 89.7 -> 0.00 mm
- net /JP1: track 86.7 -> 0.00 mm
- net /RX2: track 82.8 -> 0.00 mm, vias 2 -> 0
- net /INT2: track 73.2 -> 0.00 mm
- net /PA0: track 68.8 -> 0.00 mm
- net /PA5: track 66.3 -> 0.00 mm
- net /PF6: track 0.00 -> 56.9 mm
- net /PF5: track 0.00 -> 53.7 mm
- net /PF4: track 0.00 -> 50.8 mm
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Other:
- net class Default: clearance 0.2 -> 0.22; trace_width 0.25 -> 0.35
- rule trace_clearance: 0.2 -> 0.22
- board text removed: "ABU_ROBOCON_2018"
- board text removed: "ANT"
- board text removed: "Automatic Base"
- board text removed: "Bluetooth"
- board text removed: "TX1 RX1 GND VCC"
- board text removed: "TX2 RX2 GND VCC"
- board text removed: "UART0"
- board text removed: "UART2"

Commit message: Almost final automatic base mega + bridge
Parts:
- removed D1, D18: D_Zener, Diodes_THT:D_DO-35_SOD27_P7.62mm_Horizontal
- removed D20: LED, modFiles:LED_D3.0mm
- removed F3: Fuse, modFiles:Fuse_Holder
- removed Q2, Q3: IRF540N, modFiles:Voltage_Regulators
- removed R27: 1, modFiles:Resistor_small
- removed R36, R37: 560, modFiles:Resistor_small
- removed R38, R39: 10k, modFiles:Resistor_small
- removed R43: 330, modFiles:Resistor_small
- removed U3: Buck_5A, modFiles:Buck_Regulator
- added C12: 104, modFiles:Capacitor_Disc_Medium, F.Cu at (155.8, 96.9)
- added C14: 104, modFiles:Capacitor_Disc_Medium, F.Cu at (155.8, 91.5)
- added J24: CONN_01X01, modFiles:1_Pin, F.Cu at (135.3, 95.1)
- added J25: JST, Connectors_JST:JST_XH_B04B-XH-A_04x2.50mm_Straight, F.Cu at (173.4, 142.3)
- added J3: Compass & throwing, modFiles:Connector_DB_9, F.Cu at (164.4, 71.5)
- added R19: 330, modFiles:Resistor_small, F.Cu at (171.2, 55.6)
- C11: value 100uF -> 10uf; footprint modFiles:Capacitor_100uF -> modFiles:Capacitor_10uF
- C8: value 1000uF -> 10uf; footprint modFiles:Capacitor_1000uF -> modFiles:Capacitor_10uF
- D12: value D -> LED; footprint Diodes_THT:D_DO-27_P12.70mm_Horizontal -> modFiles:LED_D3.0mm
- J1: value GND VCC -> GND_VCC; footprint Pin_Headers:Pin_Header_Straight_2x05_Pitch2.54mm -> Pin_Headers:Pin_Header_Straight_2x03_Pitch2.54mm
- J11: value Compass -> J; footprint Connectors_JST:JST_XH_B04B-XH-A_04x2.50mm_Straight -> modFiles:Jumper
- J14: value Bluetooth -> J; footprint Pin_Headers:Pin_Header_Straight_1x06_Pitch2.54mm -> modFiles:Jumper
- J19, J21, J22: value CONN_01X02 -> J; footprint modFiles:Connector_Bornier_2 -> modFiles:Jumper
- J23: value CONN_01X02 -> BUCK+LLC; footprint modFiles:Connector_Bornier_2 -> modFiles:BUCK+LLC
- J7: value Throwing -> Conn_01x04; footprint Connectors_JST:JST_XH_B04B-XH-A_04x2.50mm_Straight -> Pin_Headers:Pin_Header_Straight_1x04_Pitch2.54mm
- J9: value I/O Pins -> I/O_PINS; footprint Pin_Headers:Pin_Header_Straight_1x08_Pitch2.54mm -> Pin_Headers:Pin_Header_Straight_1x05_Pitch2.54mm
- R1: value 1 -> 15K
- R25, R26: value 1 -> 10K
- R32, R33, R34: value R -> 10K
- moved R26 134.7 mm to (154.3, 76.9), turned to 270 degrees
- moved R25 131.6 mm to (151.2, 76.9), turned to 270 degrees
- moved J19 117.0 mm to (107.8, 148.0), turned to 90 degrees
- moved R32 87.1 mm to (136.8, 110.3), turned to 270 degrees
- moved J21 86.8 mm to (90.1, 105.7), turned to 0 degrees
- moved C8 80.2 mm to (153.4, 95.6), turned to 90 degrees
- moved J2 79.1 mm to (172.0, 136.5)
- moved J23 66.5 mm to (110.8, 82.9), turned to 0 degrees
- moved C11 58.7 mm to (153.4, 90.3), turned to 90 degrees
- moved J1 58.7 mm to (68.1, 112.6), turned to 0 degrees
- moved J7 57.9 mm to (109.6, 120.0), turned to 180 degrees
- moved C6 51.9 mm to (155.9, 69.5), turned to 90 degrees
- moved D12 51.6 mm to (153.1, 48.6), turned to 0 degrees
- moved J14 49.7 mm to (90.2, 103.1), turned to 0 degrees
- moved J4 48.0 mm to (174.2, 38.2)
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Connections:
- C11 pad 1: Net-(C11-Pad1) -> GND
- C11 pad 2: GND -> /L2
- C8 pad 1: /12Vin -> /L1
- D12 pad 1: /12Vin -> GND
- J10 pad 12: /12VVD -> /JP2
- J10 pad 13: /JP2 -> /PR3
- J11 pad 1: /3V3 -> GND
- J14 pad 1: (no net) -> GND
- J19 pad 1: /12Vin -> GND
- J21 pad 1: /12Vin -> +5V
- J22 pad 1: Net-(C11-Pad1) -> GND
- J23 pad 2: Net-(C11-Pad1) -> +12V
- J6 pad 1: /PF6 -> (no net)
- J7 pad 1: +5V -> Net-(J7-Pad1)
- J7 pad 2: /RX3 -> Net-(J7-Pad2)
- J7 pad 3: /TX3 -> Net-(J7-Pad3)
- J7 pad 4: GND -> Net-(J7-Pad4)
- R25 pad 1: GND -> +5V
- R25 pad 2: GND -> /L1
- R26 pad 2: +5V -> /L2
- R32 pad 1: +5V -> GND
- R32 pad 2: /PF6 -> /PR3o
- R33 pad 2: /PR2 -> /PR2o
- R34 pad 2: /PR1 -> /PR1o
- R42 pad 2: Net-(C9-Pad1) -> Net-(D10-Pad2)
- U1 pad 1: /TX0 -> (no net)
- U1 pad 43: /PR2 -> /PR2o
- U1 pad 45: /PR1 -> /PR1o
- U1 pad 47: (no net) -> /PR3o
- U1 pad 5: (no net) -> /L2
- U1 pad 6: (no net) -> /L1
- U1 pad A12: (no net) -> Net-(J7-Pad3)
- U1 pad A13: (no net) -> Net-(J7-Pad2)
- U1 pad A14: (no net) -> Net-(J7-Pad1)
- U1 pad A6: /PF6 -> (no net)
- U2 pad 16: /RX2 -> (no net)
- U2 pad A0: Net-(J9-Pad8) -> Net-(J9-Pad5)
- U2 pad A1: Net-(J9-Pad7) -> Net-(J9-Pad4)
- U2 pad A2: Net-(J9-Pad6) -> Net-(J9-Pad3)
- U2 pad A3: Net-(J9-Pad5) -> Net-(J9-Pad2)
- U2 pad A4: Net-(J9-Pad4) -> Net-(J9-Pad1)
- U2 pad A5: Net-(J9-Pad3) -> (no net)
- U2 pad A6: Net-(J9-Pad2) -> (no net)
- U2 pad A7: Net-(J9-Pad1) -> (no net)
Routing:
- net GND: track 65.5 -> 610.8 mm, vias 0 -> 6
- net +5V: track 120.2 -> 390.5 mm, vias 0 -> 4
- net +12V: track 100.4 -> 289.1 mm
- net /JP1: track 0.00 -> 91.8 mm, vias 0 -> 2
- net /INT5: track 14.8 -> 96.0 mm, vias 0 -> 2
- net /PA5: track 0.00 -> 73.5 mm
- net /PA0: track 0.00 -> 73.0 mm
- net /INT2: track 0.00 -> 71.2 mm
- net /RX3: track 0.00 -> 69.9 mm
- net /TX2: track 0.00 -> 67.3 mm, vias 0 -> 2
- net /TX3: track 0.00 -> 57.9 mm
- net /PF6: track 56.9 -> 0.00 mm
- net /INT: track 8.68 -> 62.0 mm
- net /RX0: track 0.00 -> 53.2 mm, vias 0 -> 2
- net /RX2: track 0.00 -> 45.0 mm, vias 0 -> 2
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Other:
- board outline added: 140.1 x 120.3 mm
- rule via_min_size: 0.4 -> 2
- board text added: "+"
- board text added: "12v"
- board text added: "5V"
- board text added: "9V"
- board text added: "ABU_ROBOCON_2018"
- board text added: "ANT"
- board text added: "AUTOMATIC BASE"
- board text added: "BUCK"
- board text added: "F0 F1 F2 F3 F4"
- board text added: "F1 F0 G G"
- board text added: "F2 F3 F4 F5 -"
- board text added: "FUSE LED"
- board text added: "K3 K4 K5 K6"
- board text added: "L2 L2 5V 3V3 SDA"
- board text added: "LLC"
- board text added: "P2 P1 P3 J2 12 G J1"
- board text added: "RESET LED"
- board text added: "RST_Jumper"
- board text added: "T3 R3 G SCL"
- board text added: "TX3 RX3"
- board text added: "V G R3 T3"
- board text removed: "- R3 T3 G"
- board text removed: "F0 F1 F2 F3 F4 F5 F6 F7"
- board text removed: "P2 P1 J2 12 12 G J1"
- board text removed: "TX3 RX3 GND VCC"
- board text removed: "VCC GND SCL SDA"
