File: pneumatic_khwappa/pneumatic_khwappa.sch (KiCad schematic (older format))
At the start: 37 parts, among them J1 bournier2, J10 Conn_02x03_Counter_Clockwise, J11 Conn_01x01, J2 inputs, J3 bournier1, J4 support, J5 bournier3, J6 Conn_01x01, J7 bournier4, J8 bournier5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

Commit message: Almost final automatic base mega + bridge
Parts:
- added J12: support, Pin_Headers:Pin_Header_Straight_2x08_Pitch2.54mm, symbol Conn_02x08_Counter_Clockwise
Connections:
- net COM is gone; now on net +12V: D10.1 (K), D2.1 (K), D4.1 (K), D6.1 (K), D8.1 (K), RL1.1, RL2.1, RL3.1, RL4.1, RL5.1, U1.9 (COM)
- no-connect marks 45 -> 61
Changed lines of the file:
@@
 	1    0    0    -1
 $EndComp
+$Comp
+L +12V #PWR020
+U 1 1 5B45F04E
+P 9770 2185
+F 0 "#PWR020" H 9770 2035 50  0001 C CNN
+F 1 "+12V" H 9770 2325 50  0000 C CNN
+F 2 "" H 9770 2185 50  0001 C CNN
+F 3 "" H 9770 2185 50  0001 C CNN
+	1    9770 2185
+	1    0    0    -1
+$EndComp
+$Comp
+L Conn_02x08_Counter_Clockwise J12
+U 1 1 5B45FB48
+P 2400 1570
+F 0 "J12" H 2450 1970 50  0000 C CNN
+F 1 "support" H 2450 1070 50  0000 C CNN
+F 2 "Pin_Headers:Pin_Header_Straight_2x08_Pitch2.54mm" H 2400 1570 50  0001 C CNN
+F 3 "" H 2400 1570 50  0001 C CNN
+	1    2400 1570
+	1    0    0    -1
+$EndComp
+NoConn ~ 2200 1270
+NoConn ~ 2200 1370
+NoConn ~ 2200 1470
+NoConn ~ 2200 1570
+NoConn ~ 2200 1670
+NoConn ~ 2200 1770
+NoConn ~ 2200 1870
+NoConn ~ 2200 1970
+NoConn ~ 2700 1970
+NoConn ~ 2700 1870
+NoConn ~ 2700 1770
+NoConn ~ 2700 1670
+NoConn ~ 2700 1570
+NoConn ~ 2700 1270
+NoConn ~ 2700 1370
+NoConn ~ 2700 1470
 $EndSCHEMATC
