File: pneumatic_khwappa/pneumatic_khwappa.kicad_pcb (KiCad board)
At the start: 2 copper layers, 37 parts, among them J1 bournier2, J10 Conn_02x03_Counter_Clockwise, J11 Conn_01x01, J2 inputs, J3 bournier1, J4 support, J5 bournier3, J6 Conn_01x01, J7 bournier4, J8 bournier5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

Commit message: Almost final automatic base mega + bridge
Parts:
- added J11: Conn_01x01, Connectors:1pin, F.Cu at (45.3, 42.8)
- added J12: support, Pin_Headers:Pin_Header_Straight_2x08_Pitch2.54mm, F.Cu at (60.9, 42.9)
- moved J11 5.46 mm to (94.2, 42.8)
- moved J8 1.57 mm to (56.7, 51.0)
- moved J7 1.43 mm to (72.5, 50.9)
- moved J5 1.38 mm to (88.6, 50.9)
Connections:
- D10 pad 1: /COM -> +12V
- D2 pad 1: /COM -> +12V
- D4 pad 1: /COM -> +12V
- D6 pad 1: /COM -> +12V
- D8 pad 1: /COM -> +12V
- J11 pad 1: Net-(J11-Pad1) -> (no net)
- J2 pad 1: Net-(J2-Pad1) -> (no net)
- J2 pad 11: Net-(J2-Pad11) -> (no net)
- J2 pad 12: Net-(J2-Pad12) -> (no net)
- J2 pad 13: Net-(J2-Pad13) -> (no net)
- J2 pad 14: Net-(J2-Pad14) -> (no net)
- J2 pad 15: Net-(J2-Pad15) -> (no net)
- J2 pad 16: Net-(J2-Pad16) -> (no net)
- J2 pad 3: Net-(J2-Pad3) -> (no net)
- J2 pad 5: Net-(J2-Pad5) -> (no net)
- J2 pad 7: Net-(J2-Pad7) -> (no net)
- J2 pad 9: Net-(J2-Pad9) -> (no net)
- J4 pad 1: Net-(J4-Pad1) -> (no net)
- J4 pad 10: Net-(J4-Pad10) -> (no net)
- J4 pad 11: Net-(J4-Pad11) -> (no net)
- J4 pad 12: Net-(J4-Pad12) -> (no net)
- J4 pad 13: Net-(J4-Pad13) -> (no net)
- J4 pad 14: Net-(J4-Pad14) -> (no net)
- J4 pad 15: Net-(J4-Pad15) -> (no net)
- J4 pad 16: Net-(J4-Pad16) -> (no net)
- J4 pad 17: Net-(J4-Pad17) -> (no net)
- J4 pad 18: Net-(J4-Pad18) -> (no net)
- J4 pad 19: Net-(J4-Pad19) -> (no net)
- J4 pad 2: Net-(J4-Pad2) -> (no net)
- J4 pad 20: Net-(J4-Pad20) -> (no net)
- J4 pad 21: Net-(J4-Pad21) -> (no net)
- J4 pad 22: Net-(J4-Pad22) -> (no net)
- J4 pad 23: Net-(J4-Pad23) -> (no net)
- J4 pad 24: Net-(J4-Pad24) -> (no net)
- J4 pad 25: Net-(J4-Pad25) -> (no net)
- J4 pad 26: Net-(J4-Pad26) -> (no net)
- J4 pad 27: Net-(J4-Pad27) -> (no net)
- J4 pad 28: Net-(J4-Pad28) -> (no net)
- J4 pad 29: Net-(J4-Pad29) -> (no net)
- J4 pad 3: Net-(J4-Pad3) -> (no net)
- J4 pad 30: Net-(J4-Pad30) -> (no net)
- J4 pad 4: Net-(J4-Pad4) -> (no net)
- J4 pad 5: Net-(J4-Pad5) -> (no net)
- J4 pad 6: Net-(J4-Pad6) -> (no net)
- J4 pad 7: Net-(J4-Pad7) -> (no net)
- J4 pad 8: Net-(J4-Pad8) -> (no net)
- J4 pad 9: Net-(J4-Pad9) -> (no net)
- J6 pad 1: Net-(J6-Pad1) -> (no net)
- RL1 pad 1: /COM -> +12V
- RL2 pad 1: /COM -> +12V
- RL3 pad 1: /COM -> +12V
- RL4 pad 1: /COM -> +12V
- RL5 pad 1: /COM -> +12V
- U1 pad 10: Net-(U1-Pad10) -> (no net)
- U1 pad 6: Net-(U1-Pad6) -> (no net)
- U1 pad 7: Net-(U1-Pad7) -> (no net)
- U1 pad 9: /COM -> +12V
Routing:
- net (no net): track 302.8 -> 0.00 mm
- net +12V: track 148.7 -> 367.0 mm
- net /COM: track 212.4 -> 0.00 mm
- net GND: track 0.69 -> 14.0 mm
- net /NO5: track 14.8 -> 13.2 mm
- net /NO4: track 16.0 -> 14.5 mm
- net /NO3: track 16.8 -> 15.4 mm
Other:
- board text added: "ABU ROBOCON 2018"
- board text added: "SAM"

Commit message: Final for ABU_ROBOCON_2018 Automatic_Base
Parts:
- moved J11 80.9 mm to (116.6, 120.5), turned to 0 degrees
- moved J11 76.9 mm to (116.6, 71.6), turned to 0 degrees
- moved J12 71.1 mm to (116.5, 87.2), turned to 0 degrees
- moved J6 69.4 mm to (22.2, 71.8), turned to 0 degrees
- moved D9 67.0 mm to (109.6, 73.0), turned to 180 degrees
- moved J5 67.0 mm to (108.4, 114.9), turned to 90 degrees
- moved J2 65.5 mm to (21.7, 81.2), turned to 0 degrees
- moved C3 63.4 mm to (102.0, 120.3), turned to 90 degrees
- moved D5 63.0 mm to (109.6, 104.3), turned to 180 degrees
- moved D7 61.2 mm to (109.6, 88.5), turned to 180 degrees
- moved J8 60.7 mm to (108.4, 83.0), turned to 90 degrees
- moved J7 59.8 mm to (108.4, 98.7), turned to 90 degrees
- moved J9 59.8 mm to (29.3, 112.9), turned to 180 degrees
- moved R3 57.6 mm to (102.0, 112.9), turned to 90 degrees
- moved U1 57.6 mm to (27.6, 81.2), turned to 0 degrees
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Routing:
- net (no net): track 0.00 -> 314.2 mm
