File: Automatic3.0/Power/Power_Supply.sch (KiCad schematic (older format))
At the start: 35 parts, among them J16 CONN_01X02, J17 Reset_Jumper, J18 Reset_Jumper, SW1 Reset, SW2 Reset, U4 LM7809, U5 Buck

Commit message: Final for ABU_ROBOCON_2018 Automatic_Base
Parts:
- D13: value LED_5V -> MEGA_OUT
- D19: value LED_5V -> MEGA OUT
- D6, D7: value LED_9V -> MEGA_IN
- D8: value LED_5V -> BUCK_OUT
- D9: value LED_BUCK -> BUCK_IN
Changed lines of the file:
@@
 $EndDescr
 $Comp
-L +12V #PWR041
+L +12V #PWR043
 U 1 1 5ADD8405
 P 1400 1225
-F 0 "#PWR041" H 1400 1075 50  0001 C CNN
+F 0 "#PWR043" H 1400 1075 50  0001 C CNN
 F 1 "+12V" H 1400 1365 50  0000 C CNN
 F 2 "" H 1400 1225 50  0001 C CNN
@@
 P 3250 1350
 F 0 "D8" H 3250 1450 50  0000 C CNN
-F 1 "LED_5V" H 3250 1250 50  0000 C CNN
+F 1 "BUCK_OUT" H 3250 1250 50  0000 C CNN
 F 2 "modFiles:LED_D3.0mm" H 3250 1350 50  0001 C CNN
 F 3 "" H 3250 1350 50  0001 C CNN
@@
 $EndComp
 $Comp
-L GND #PWR042
+L GND #PWR044
 U 1 1 5ADD84AA
 P 3475 1400
-F 0 "#PWR042" H 3475 1150 50  0001 C CNN
+F 0 "#PWR044" H 3475 1150 50  0001 C CNN
 F 1 "GND" H 3475 1250 50  0000 C CNN
 F 2 "" H 3475 1400 50  0001 C CNN
@@
 P 3275 1900
 F 0 "D9" H 3275 2000 50  0000 C CNN
-F 1 "LED_BUCK" H 3275 1800 50  0000 C CNN
+F 1 "BUCK_IN" H 3275 1800 50  0000 C CNN
 F 2 "modFiles:LED_D3.0mm" H 3275 1900 50  0001 C CNN
 F 3 "" H 3275 1900 50  0001 C CNN
@@
 $EndComp
 $Comp
-L GND #PWR043
+L GND #PWR045
 U 1 1 5ADD8645
 P 3500 1950
-F 0 "#PWR043" H 3500 1700 50  0001 C CNN
+F 0 "#PWR045" H 3500 1700 50  0001 C CNN
 F 1 "GND" H 3500 1800 50  0000 C CNN
 F 2 "" H 3500 1950 50  0001 C CNN
@@
 $EndComp
 $Comp
-L GND #PWR044
+L GND #PWR046
 U 1 1 5ADD88DA
 P 2200 1375
-F 0 "#PWR044" H 2200 1125 50  0001 C CNN
+F 0 "#PWR046" H 2200 1125 50  0001 C CNN
 F 1 "GND" H 2200 1225 50  0000 C CNN
 F 2 "" H 2200 1375 50  0001 C CNN
@@
 P 2000 1875
 F 0 "D6" H 2000 1975 50  0000 C CNN
-F 1 "LED_9V" H 2000 1775 50  0000 C CNN
+F 1 "MEGA_IN" H 2000 1775 50  0000 C CNN
 F 2 "modFiles:LED_D3.0mm" H 2000 1875 50  0001 C CNN
 F 3 "" H 2000 1875 50  0001 C CNN
@@
 $EndComp
 $Comp
-L GND #PWR045
+L GND #PWR047
 U 1 1 5ADD88F7
 P 2225 1925
-F 0 "#PWR045" H 2225 1675 50  0001 C CNN
+F 0 "#PWR047" H 2225 1675 50  0001 C CNN
 F 1 "GND" H 2225 1775 50  0000 C CNN
 F 2 "" H 2225 1925 50  0001 C CNN
@@
 $EndComp
 $Comp
-L +9V #PWR046
+L +9V #PWR048
 U 1 1 5ADD8969
 P 1425 1775
-F 0 "#PWR046" H 1425 1625 50  0001 C CNN
+F 0 "#PWR048" H 1425 1625 50  0001 C CNN
 F 1 "+9V" H 1425 1915 50  0000 C CNN
 F 2 "" H 1425 1775 50  0001 C CNN
@@
 $EndComp
 $Comp
-L +5V #PWR047
+L +5V #PWR049
 U 1 1 5ADD89A5
 P 2675 1250
-F 0 "#PWR047" H 2675 1100 50  0001 C CNN
+F 0 "#PWR049" H 2675 1100 50  0001 C CNN
 F 1 "+5V" H 2675 1390 50  0000 C CNN
 F 2 "" H 2675 1250 50  0001 C CNN
@@
 $EndComp
 $Comp
-L +12V #PWR048
+L +12V #PWR050
 U 1 1 5ADD8D0E
 P 2600 3225
-F 0 "#PWR048" H 2600 3075 50  0001 C CNN
+F 0 "#PWR050" H 2600 3075 50  0001 C CNN
 F 1 "+12V" H 2600 3365 50  0000 C CNN
 F 2 "" H 2600 3225 50  0001 C CNN
@@
 $EndComp
 $Comp
-L +9V #PWR049
+L +9V #PWR051
 U 1 1 5ADD8DBB
 P 4850 3225
-F 0 "#PWR049" H 4850 3075 50  0001 C CNN
+F 0 "#PWR051" H 4850 3075 50  0001 C CNN
 F 1 "+9V" H 4850 3365 50  0000 C CNN
 F 2 "" H 4850 3225 50  0001 C CNN
@@
 POWER_FOR_MEGA
 $Comp
-L GND #PWR050
+L GND #PWR052
 U 1 1 5ADD935A
 P 4125 3800
-F 0 "#PWR050" H 4125 3550 50  0001 C CNN
+F 0 "#PWR052" H 4125 3550 50  0001 C CNN
 F 1 "GND" H 4125 3650 50  0000 C CNN
 F 2 "" H 4125 3800 50  0001 C CNN
@@
 $EndComp
 $Comp
-L +12V #PWR051
+L +12V #PWR053
 U 1 1 5ADDD1E7
 P 1690 4465
-F 0 "#PWR051" H 1690 4315 50  0001 C CNN
+F 0 "#PWR053" H 1690 4315 50  0001 C CNN
 F 1 "+12V" H 1690 4605 50  0000 C CNN
 F 2 "" H 1690 4465 50  0001 C CNN
@@
 $EndComp
 $Comp
-L GND #PWR052
+L GND #PWR054
 U 1 1 5ADDD3BB
 P 1690 4615
-F 0 "#PWR052" H 1690 4365 50  0001 C CNN
+F 0 "#PWR054" H 1690 4365 50  0001 C CNN
 F 1 "GND" H 1690 4465 50  0000 C CNN
 F 2 "" H 1690 4615 50  0001 C CNN
@@
 P 4475 1850
 F 0 "D13" H 4475 1950 50  0000 C CNN
-F 1 "LED_5V" H 4475 1750 50  0000 C CNN
+F 1 "MEGA_OUT" H 4475 1750 50  0000 C CNN
 F 2 "modFiles:LED_D3.0mm" H 4475 1850 50  0001 C CNN
 F 3 "" H 4475 1850 50  0001 C CNN
@@
 $EndComp
 $Comp
-L GND #PWR053
+L GND #PWR055
 U 1 1 5B14130A
 P 4700 1900
-F 0 "#PWR053" H 4700 1650 50  0001 C CNN
+F 0 "#PWR055" H 4700 1650 50  0001 C CNN
 F 1 "GND" H 4700 1750 50  0000 C CNN
 F 2 "" H 4700 1900 50  0001 C CNN
@@
 $EndComp
 $Comp
-L GND #PWR054
+L GND #PWR056
 U 1 1 5B1417E4
 P 8075 1925
-F 0 "#PWR054" H 8075 1675 50  0001 C CNN
+F 0 "#PWR056" H 8075 1675 50  0001 C CNN
 F 1 "GND" H 8075 1775 50  0000 C CNN
 F 2 "" H 8075 1925 50  0001 C CNN
@@
 3V3
 $Comp
-L GND #PWR055
+L GND #PWR057
 U 1 1 5B14194B
 P 8625 1375
-F 0 "#PWR055" H 8625 1125 50  0001 C CNN
+F 0 "#PWR057" H 8625 1125 50  0001 C CNN
 F 1 "GND" H 8625 1225 50  0000 C CNN
 F 2 "" H 8625 1375 50  0001 C CNN
@@
 $EndComp
 $Comp
-L GND #PWR056
+L GND #PWR058
 U 1 1 5B142045
 P 6700 1925
-F 0 "#PWR056" H 6700 1675 50  0001 C CNN
+F 0 "#PWR058" H 6700 1675 50  0001 C CNN
 F 1 "GND" H 6700 1775 50  0000 C CNN
 F 2 "" H 6700 1925 50  0001 C CNN
@@
 5V
 $Comp
-L GND #PWR057
+L GND #PWR059
 U 1 1 5B14204C
 P 7250 1375
-F 0 "#PWR057" H 7250 1125 50  0001 C CNN
+F 0 "#PWR059" H 7250 1125 50  0001 C CNN
 F 1 "GND" H 7250 1225 50  0000 C CNN
 F 2 "" H 7250 1375 50  0001 C CNN
@@
 P 2025 2450
 F 0 "D7" H 2025 2550 50  0000 C CNN
-F 1 "LED_9V" H 2025 2350 50  0000 C CNN
+F 1 "MEGA_IN" H 2025 2350 50  0000 C CNN
 F 2 "modFiles:LED_D3.0mm" H 2025 2450 50  0001 C CNN
 F 3 "" H 2025 2450 50  0001 C CNN
@@
 $EndComp
 $Comp
-L GND #PWR058
+L GND #PWR060
 U 1 1 5B14315F
 P 2250 2500
-F 0 "#PWR058" H 2250 2250 50  0001 C CNN
+F 0 "#PWR060" H 2250 2250 50  0001 C CNN
 F 1 "GND" H 2250 2350 50  0000 C CNN
 F 2 "" H 2250 2500 50  0001 C CNN
@@
 $EndComp
 $Comp
-L +9V #PWR059
+L +9V #PWR061
 U 1 1 5B143165
 P 1450 2350
-F 0 "#PWR059" H 1450 2200 50  0001 C CNN
+F 0 "#PWR061" H 1450 2200 50  0001 C CNN
 F 1 "+9V" H 1450 2490 50  0000 C CNN
 F 2 "" H 1450 2350 50  0001 C CNN
@@
 R1
 $Comp
-L +12V #PWR060
+L +12V #PWR062
 U 1 1 5B40FCE5
 P 1850 5550
-F 0 "#PWR060" H 1850 5400 50  0001 C CNN
+F 0 "#PWR062" H 1850 5400 50  0001 C CNN
 F 1 "+12V" H 1850 5690 50  0000 C CNN
 F 2 "" H 1850 5550 50  0001 C CNN
@@
 $EndComp
 $Comp
-L GND #PWR061
+L GND #PWR063
 U 1 1 5B40FD03
 P 3800 6450
-F 0 "#PWR061" H 3800 6200 50  0001 C CNN
+F 0 "#PWR063" H 3800 6200 50  0001 C CNN
 F 1 "GND" H 3800 6300 50  0000 C CNN
 F 2 "" H 3800 6450 50  0001 C CNN
@@
 $EndComp
 $Comp
-L +5V #PWR062
+L +5V #PWR064
 U 1 1 5B40FD09
 P 4550 5660
-F 0 "#PWR062" H 4550 5510 50  0001 C CNN
+F 0 "#PWR064" H 4550 5510 50  0001 C CNN
 F 1 "+5V" H 4550 5800 50  0000 C CNN
 F 2 "" H 4550 5660 50  0001 C CNN
@@
 P 5950 1800
 F 0 "D19" H 5950 1900 50  0000 C CNN
-F 1 "LED_5V" H 5950 1700 50  0000 C CNN
+F 1 "MEGA OUT" H 5950 1700 50  0000 C CNN
 F 2 "modFiles:LED_D3.0mm" H 5950 1800 50  0001 C CNN
 F 3 "" H 5950 1800 50  0001 C CNN
@@
 $EndComp
 $Comp
-L GND #PWR063
+L GND #PWR065
 U 1 1 5B3FFCF9
 P 6175 1850
-F 0 "#PWR063" H 6175 1600 50  0001 C CNN
+F 0 "#PWR065" H 6175 1600 50  0001 C CNN
 F 1 "GND" H 6175 1700 50  0000 C CNN
 F 2 "" H 6175 1850 50  0001 C CNN
@@
 	3125 2830 3125 2870
 $Comp
-L GND #PWR064
+L GND #PWR066
 U 1 1 5B425818
 P 3385 2530
-F 0 "#PWR064" H 3385 2280 50  0001 C CNN
+F 0 "#PWR066" H 3385 2280 50  0001 C CNN
 F 1 "GND" H 3385 2380 50  0000 C CNN
 F 2 "" H 3385 2530 50  0001 C CNN
@@
 	2400 5235 2400 5275
 $Comp
-L GND #PWR065
+L GND #PWR067
 U 1 1 5B4694A6
 P 2660 4935
-F 0 "#PWR065" H 2660 4685 50  0001 C CNN
+F 0 "#PWR067" H 2660 4685 50  0001 C CNN
 F 1 "GND" H 2660 4785 50  0000 C CNN
 F 2 "" H 2660 4935 50  0001 C CNN
