File: mannual/LED/LED.kicad_pcb (KiCad board)
At the start: 2 copper layers, 20 parts, among them J1 Conn_01x06, J2 Conn_01x07

Commit message: Final for ABU_ROBOCON_2018 Automatic_Base
Parts:
- added 330: R, test:Resistor_small, F.Cu at (161.2, 41.3)
- added 330: R, test:Resistor_small, F.Cu at (253.4, 46.7)
- added 330: R, test:Resistor_small, F.Cu at (253.4, 38.6)
- added 330: R, test:Resistor_small, F.Cu at (253.4, 41.3)
- added 330: R, test:Resistor_small, F.Cu at (161.2, 38.6)
- added 330: R, test:Resistor_small, F.Cu at (161.2, 46.7)
- added 330: R, test:Resistor_small, F.Cu at (161.2, 44.0)
- added 330: R, test:Resistor_small, F.Cu at (161.2, 35.8)
- added 330: R, test:Resistor_small, F.Cu at (161.2, 33.1)
- added 330: R, test:Resistor_small, F.Cu at (253.4, 33.1)
- added 330: R, test:Resistor_small, F.Cu at (253.4, 35.8)
- added 330: R, test:Resistor_small, F.Cu at (253.4, 44.0)
- added C1: C, modFiles:Capacitor_10uF, F.Cu at (158.3, 26.9)
- added C1: C, modFiles:Capacitor_10uF, F.Cu at (250.5, 26.9)
- added C2: C, modFiles:Capacitor_10uF, F.Cu at (146.9, 51.8)
- added C2: C, modFiles:Capacitor_10uF, F.Cu at (239.1, 51.8)
- added C3: C, modFiles:Capacitor_10uF, F.Cu at (149.2, 26.9)
- added C3: C, modFiles:Capacitor_10uF, F.Cu at (241.4, 26.9)
- added C4: C, modFiles:Capacitor_10uF, F.Cu at (152.6, 26.9)
- added C4: C, modFiles:Capacitor_10uF, F.Cu at (244.8, 26.9)
- added C5: C, modFiles:Capacitor_10uF, F.Cu at (152.6, 51.8)
- added C5: C, modFiles:Capacitor_10uF, F.Cu at (244.8, 51.8)
- added C6: C, modFiles:Capacitor_10uF, F.Cu at (158.4, 51.8)
- added C6: C, modFiles:Capacitor_10uF, F.Cu at (250.6, 51.8)
- added D1: LED, LEDs:LED_Rectangular_W5.0mm_H2.0mm, F.Cu at (152.1, 41.3)
- added D1: LED, LEDs:LED_Rectangular_W5.0mm_H2.0mm, F.Cu at (244.3, 41.3)
- added D2: LED, LEDs:LED_Rectangular_W5.0mm_H2.0mm, F.Cu at (152.1, 38.6)
- added D2: LED, LEDs:LED_Rectangular_W5.0mm_H2.0mm, F.Cu at (244.3, 38.6)
- added D3: LED, LEDs:LED_Rectangular_W5.0mm_H2.0mm, F.Cu at (152.1, 46.7)
- added D3: LED, LEDs:LED_Rectangular_W5.0mm_H2.0mm, F.Cu at (244.3, 46.7)
- added D4: LED, LEDs:LED_Rectangular_W5.0mm_H2.0mm, F.Cu at (152.1, 44.0)
- added D4: LED, LEDs:LED_Rectangular_W5.0mm_H2.0mm, F.Cu at (244.3, 44.0)
- added D5: LED, LEDs:LED_Rectangular_W5.0mm_H2.0mm, F.Cu at (152.1, 35.8)
- added D5: LED, LEDs:LED_Rectangular_W5.0mm_H2.0mm, F.Cu at (244.3, 35.8)
- added D6: LED, LEDs:LED_Rectangular_W5.0mm_H2.0mm, F.Cu at (152.1, 33.1)
- added D6: LED, LEDs:LED_Rectangular_W5.0mm_H2.0mm, F.Cu at (244.3, 33.1)
- added J1: Conn_01x06, Pin_Headers:Pin_Header_Straight_1x06_Pitch2.54mm, F.Cu at (146.1, 33.5)
- added J1: Conn_01x06, Pin_Headers:Pin_Header_Straight_1x06_Pitch2.54mm, F.Cu at (238.3, 33.5)
- added J2: Conn_01x07, Pin_Headers:Pin_Header_Straight_1x07_Pitch2.54mm, F.Cu at (163.1, 46.8)
- added J2: Conn_01x07, Pin_Headers:Pin_Header_Straight_1x07_Pitch2.54mm, F.Cu at (255.3, 46.8)
- moved C1 2.12 mm to (68.4, 27.6)
- moved C6 1.94 mm to (68.4, 52.5)
- moved C4 1.22 mm to (62.6, 27.7)
- moved C5 1.16 mm to (62.7, 52.5)
- moved C2 0.17 mm to (56.9, 52.5)
- moved C3 0.17 mm to (59.3, 27.6)
- renumbered 10K to 330
Routing:
- net (no net): track 207.2 -> 607.2 mm
- net Net-(C1-Pad2): track 89.1 -> 258.6 mm
- net Net-(C2-Pad2): track 23.0 -> 69.7 mm
- net Net-(C3-Pad1): track 24.2 -> 70.9 mm
- net Net-(C4-Pad2): track 14.7 -> 45.5 mm
- net Net-(C5-Pad2): track 13.4 -> 43.3 mm
- net Net-(C1-Pad1): track 9.59 -> 31.1 mm
- net Net-(C6-Pad2): track 7.85 -> 24.1 mm
- net Net-(D6-Pad2): track 3.69 -> 11.1 mm
- net Net-(D3-Pad2): track 3.69 -> 11.1 mm
- net Net-(D4-Pad2): track 3.63 -> 10.9 mm
- net Net-(D5-Pad2): track 3.61 -> 10.8 mm
- net Net-(D1-Pad2): track 3.57 -> 10.7 mm
- net Net-(D2-Pad2): track 3.53 -> 10.6 mm
- net Net-(D5-Pad1): track 2.40 -> 7.19 mm
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