File: Automatic3.0/Buck+LLC/Buck.sch (KiCad schematic (older format))
At the start: 29 parts, among them J1 OUT, J2 LED, J3 LED, J4 Conn_01x12, J5 LM324, J6 LED, J7 Conn_01x01, J8 Conn_01x01, Q1 TIP122, Q2 TIP122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

Commit message: Buck circuit also modified and pdfs also changed
Parts:
- removed J5: LM324, Housings_DIP:DIP-14_W7.62mm, symbol Conn_02x07_Counter_Clockwise
- removed R6, R7: R, modFiles:Resistor_small, symbol R
- added D3, D4, D5: D, modFiles:Diode_small, symbol D
- R10, R8, R9: value 10k -> 39k
- R11, R2, R4: value 2K2 -> 3k3
Connections:
- net labels removed: IN1+, IN1-, IN2+, IN2-, IN3+, IN3-, IN4+, IN4-, OUT1, OUT2, OUT3, OUT4
- wire segments 66 -> 51
Changed lines of the file:
@@
 P 6925 3675
 F 0 "R2" V 7005 3675 50  0000 C CNN
-F 1 "2K2" V 6925 3675 50  0000 C CNN
+F 1 "3k3" V 6925 3675 50  0000 C CNN
 F 2 "modFiles:Resistor_small" V 6855 3675 50  0001 C CNN
 F 3 "" H 6925 3675 50  0001 C CNN
@@
 P 8300 3675
 F 0 "R4" V 8380 3675 50  0000 C CNN
-F 1 "2K2" V 8300 3675 50  0000 C CNN
+F 1 "3k3" V 8300 3675 50  0000 C CNN
 F 2 "modFiles:Resistor_small" V 8230 3675 50  0001 C CNN
 F 3 "" H 8300 3675 50  0001 C CNN
@@
 $EndComp
 $Comp
-L Conn_02x07_Counter_Clockwise J5
-U 1 1 5B490223
-P 2275 4725
-F 0 "J5" H 2325 5125 50  0000 C CNN
-F 1 "LM324" H 2325 4325 50  0000 C CNN
-F 2 "Housings_DIP:DIP-14_W7.62mm" H 2275 4725 50  0001 C CNN
-F 3 "" H 2275 4725 50  0001 C CNN
-	1    2275 4725
-	1    0    0    -1
-$EndComp
-$Comp
-L +5V #PWR06
-U 1 1 5B4903B2
-P 2075 4725
-F 0 "#PWR06" H 2075 4575 50  0001 C CNN
-F 1 "+5V" H 2075 4865 50  0000 C CNN
-F 2 "" H 2075 4725 50  0001 C CNN
-F 3 "" H 2075 4725 50  0001 C CNN
-	1    2075 4725
-	0    -1   -1   0
-$EndComp
-$Comp
-L GND #PWR07
-U 1 1 5B4903F0
-P 2575 4725
-F 0 "#PWR07" H 2575 4475 50  0001 C CNN
-F 1 "GND" H 2575 4575 50  0000 C CNN
-F 2 "" H 2575 4725 50  0001 C CNN
-F 3 "" H 2575 4725 50  0001 C CNN
-	1    2575 4725
-	0    -1   -1   0
-$EndComp
-Text Label 2075 4525 2    60   ~ 0
-IN1-
-Text Label 2075 5025 2    60   ~ 0
-OUT2
-Text Label 2075 4925 2    60   ~ 0
-IN2-
-Text Label 2575 4425 0    60   ~ 0
-OUT4
-Text Label 2575 4525 0    60   ~ 0
-IN4-
-Text Label 2575 5025 0    60   ~ 0
-OUT3
-Text Label 2575 4925 0    60   ~ 0
-IN3-
-Text Label 7175 875  0    60   ~ 0
-IN1-
-$Comp
-L GND #PWR08
-U 1 1 5B4917AD
-P 6875 1100
-F 0 "#PWR08" H 6875 850 50  0001 C CNN
-F 1 "GND" H 6875 950 50  0000 C CNN
-F 2 "" H 6875 1100 50  0001 C CNN
-F 3 "" H 6875 1100 50  0001 C CNN
-	1    6875 1100
-	1    0    0    -1
-$EndComp
-$Comp
-L +12V #PWR09
+L +12V #PWR06
 U 1 1 5B49CF5D
 P 2175 2125
-F 0 "#PWR09" H 2175 1975 50  0001 C CNN
+F 0 "#PWR06" H 2175 1975 50  0001 C CNN
 F 1 "+12V" H 2175 2265 50  0000 C CNN
 F 2 "" H 2175 2125 50  0001 C CNN
@@
 $EndComp
 $Comp
-L GND #PWR010
+L GND #PWR07
 U 1 1 5B49D143
 P 1950 2025
-F 0 "#PWR010" H 1950 1775 50  0001 C CNN
+F 0 "#PWR07" H 1950 1775 50  0001 C CNN
 F 1 "GND" H 1950 1875 50  0000 C CNN
 F 2 "" H 1950 2025 50  0001 C CNN
@@
 $EndComp
 $Comp
-L +5V #PWR011
+L +5V #PWR08
 U 1 1 5B49D34F
 P 1950 2225
-F 0 "#PWR011" H 1950 2075 50  0001 C CNN
+F 0 "#PWR08" H 1950 2075 50  0001 C CNN
 F 1 "+5V" H 1950 2365 50  0000 C CNN
 F 2 "" H 1950 2225 50  0001 C CNN
@@
 	0    1    1    0
 $EndComp
-$Comp
-L R R7
-U 1 1 5B4A2A6C
-P 7025 1025
-F 0 "R7" V 7105 1025 50  0000 C CNN
-F 1 "R" V 7025 1025 50  0000 C CNN
-F 2 "modFiles:Resistor_small" V 6955 1025 50  0001 C CNN
-F 3 "" H 7025 1025 50  0001 C CNN
-	1    7025 1025
-	0    1    1    0
-$EndComp
-$Comp
-L R R6
-U 1 1 5B4A2A13
-P 7025 875
-F 0 "R6" V 7105 875 50  0000 C CNN
-F 1 "R" V 7025 875 50  0000 C CNN
-F 2 "modFiles:Resistor_small" V 6955 875 50  0001 C CNN
-F 3 "" H 7025 875 50  0001 C CNN
-	1    7025 875
-	0    1    1    0
-$EndComp
+Text Label 1950 2325 0    60   ~ 0
+PR1
+Text Label 1950 2425 0    60   ~ 0
+PR2
 Text Label 1950 2525 0    60   ~ 0
-PR1
-Text Label 1950 2325 0    60   ~ 0
-PR2
-Text Label 1950 2425 0    60   ~ 0
 PR3
+Text Label 1950 2625 0    60   ~ 0
+PR1o
+Text Label 1950 2725 0    60   ~ 0
+PR2o
 Text Label 1950 2825 0    60   ~ 0
-PR1o
-Text Label 1950 2625 0    60   ~ 0
-PR2o
-Text Label 1950 2725 0    60   ~ 0
 PR3o
 Text Label 1950 2925 0    60   ~ 0
@@
 Text Label 1950 3025 0    60   ~ 0
 LED2
-Text Label 1575 4625 0    60   ~ 0
+Text Label 4150 4875 2    60   ~ 0
 PR1
-Text Label 1575 4825 0    60   ~ 0
+Text Label 4150 5200 2    60   ~ 0
 PR2
 Text Label 4325 3325 3    60   ~ 0
 PR3
-Text Label 1575 4425 0    60   ~ 0
+Text Label 4450 4875 0    60   ~ 0
 PR1o
-Text Label 1575 5025 0    60   ~ 0
+Text Label 4450 5200 0    60   ~ 0
 PR2o
-Text Label 2900 5025 0    60   ~ 0
+Text Label 4475 4550 0    60   ~ 0
 PR3o
-Text Label 2075 4825 2    60   ~ 0
-IN2+
-Text Label 2575 4825 0    60   ~ 0
-IN3+
-Text Label 2575 4625 0    60   ~ 0
-IN4+
-Text Label 2075 4625 2    60   ~ 0
-IN1+
-Text Label 2075 4425 2    60   ~ 0
-OUT1
 Text Label 6775 3675 2    60   ~ 0
 LED1
@@
 Connection ~ 7475 1975
 Wire Wire Line
-	2075 4925 2575 4925
-Wire Wire Line
-	2325 4925 2325 4525
-Connection ~ 2325 4925
-Wire Wire Line
-	2325 4525 2075 4525
-Wire Wire Line
 	2175 2125 1950 2125
-Wire Wire Line
-	7175 875  7175 1025
-Wire Wire Line
-	6875 1025 6875 1100
 Wire Wire Line
 	4675 1650 4675 2850
@@
 Wire Wire Line
 	4675 1975 8850 1975
-Wire Wire Line
-	2075 4425 1575 4425
-Wire Wire Line
-	1575 4625 2075 4625
-Wire Wire Line
-	1575 4825 2075 4825
-Wire Wire Line
-	2075 5025 1575 5025
-Wire Wire Line
-	2575 4825 2900 4825
-Wire Wire Line
-	2900 5025 2575 5025
-Wire Wire Line
-	6050 875  6875 875
-Wire Wire Line
-	9025 1975 9025 1900
 $Comp
 L Conn_01x01 J7
@@
 P 4750 3175
 F 0 "R8" V 4830 3175 50  0000 C CNN
-F 1 "10k" V 4750 3175 50  0000 C CNN
+F 1 "39k" V 4750 3175 50  0000 C CNN
 F 2 "modFiles:Resistor_small" V 4680 3175 50  0001 C CNN
 F 3 "" H 4750 3175 50  0001 C CNN
@@
 P 4525 3175
 F 0 "R9" V 4605 3175 50  0000 C CNN
-F 1 "10k" V 4525 3175 50  0000 C CNN
+F 1 "39k" V 4525 3175 50  0000 C CNN
 F 2 "modFiles:Resistor_small" V 4455 3175 50  0001 C CNN
 F 3 "" H 4525 3175 50  0001 C CNN
@@
 P 4325 3175
 F 0 "R10" V 4405 3175 50  0000 C CNN
-F 1 "10k" V 4325 3175 50  0000 C CNN
+F 1 "39k" V 4325 3175 50  0000 C CNN
 F 2 "modFiles:Resistor_small" V 4255 3175 50  0001 C CNN
 F 3 "" H 4325 3175 50  0001 C CNN
@@
 $EndComp
 Wire Wire Line
-	4525 2975 4750 2975
+	4325 2975 4750 2975
 Wire Wire Line
 	4750 2975 4750 3025
@@
 	4525 2975 4525 3025
 Connection ~ 4625 2975
-$Comp
-L GND #PWR012
-U 1 1 5B561CAE
-P 4325 3025
-F 0 "#PWR012" H 4325 2775 50  0001 C CNN
-F 1 "GND" H 4325 2875 50  0000 C CNN
-F 2 "" H 4325 3025 50  0001 C CNN
-F 3 "" H 4325 3025 50  0001 C CNN
-	1    4325 3025
-	-1   0    0    1
-$EndComp
 Text Label 4750 3325 3    60   ~ 0
 PR1
 Text Label 4525 3325 3    60   ~ 0
 PR2
-Text Label 2900 4825 0    60   ~ 0
+Text Label 4175 4550 2    60   ~ 0
 PR3
-Connection ~ 6875 1075
-Connection ~ 9025 1900
 Connection ~ 8850 1975
 Wire Wire Line
@@
 P 9750 3775
 F 0 "R11" V 9830 3775 50  0000 C CNN
-F 1 "2K2" V 9750 3775 50  0000 C CNN
+F 1 "3k3" V 9750 3775 50  0000 C CNN
 F 2 "modFiles:Resistor_small" V 9680 3775 50  0001 C CNN
 F 3 "" H 9750 3775 50  0001 C CNN
@@
 $EndComp
 $Comp
-L GND #PWR013
+L GND #PWR09
 U 1 1 5B5CFAFF
 P 10250 4250
-F 0 "#PWR013" H 10250 4000 50  0001 C CNN
+F 0 "#PWR09" H 10250 4000 50  0001 C CNN
 F 1 "GND" H 10250 4100 50  0000 C CNN
 F 2 "" H 10250 4250 50  0001 C CNN
@@
 Wire Wire Line
 	10300 3400 10250 3400
-Wire Wire Line
-	10250 3400 10250 3575
 Wire Wire Line
 	9900 3775 9950 3775
@@
 	5025 2250 5025 1950
 Connection ~ 4675 1975
-Wire Wire Line
-	6050 875  6050 1950
-Wire Wire Line
-	6050 1950 5025 1950
+Connection ~ 10250 3550
+$Comp
+L D D3
+U 1 1 5B67F017
+P 4300 4875
+F 0 "D3" H 4300 4975 50  0000 C CNN
+F 1 "D" H 4300 4775 50  0000 C CNN
+F 2 "modFiles:Diode_small" H 4300 4875 50  0001 C CNN
+F 3 "" H 4300 4875 50  0001 C CNN
+	1    4300 4875
+	1    0    0    -1
+$EndComp
+$Comp
+L D D5
+U 1 1 5B67F09E
+P 4325 4550
+F 0 "D5" H 4325 4650 50  0000 C CNN
+F 1 "D" H 4325 4450 50  0000 C CNN
+F 2 "modFiles:Diode_small" H 4325 4550 50  0001 C CNN
+F 3 "" H 4325 4550 50  0001 C CNN
+	1    4325 4550
+	1    0    0    -1
+$EndComp
+$Comp
+L D D4
+U 1 1 5B67F13B
+P 4300 5200
+F 0 "D4" H 4300 5300 50  0000 C CNN
+F 1 "D" H 4300 5100 50  0000 C CNN
+F 2 "modFiles:Diode_small" H 4300 5200 50  0001 C CNN
+F 3 "" H 4300 5200 50  0001 C CNN
+	1    4300 5200
+	1    0    0    -1
+$EndComp
+Wire Wire Line
+	4325 2975 4325 3025
+Connection ~ 4525 2975
 $EndSCHEMATC
