File: debugger/Debugger.sch (KiCad schematic (older format))
At the start: 176 parts, among them J1 CONN_01X02, J10 DB9_FEMALE, J11 DB25_FEMALE, J12 USB_A, J13 USB_B, J14 RJ45, J2 DB15_FEMALE, J3 DB15_FEMALE, J4 CONN_01X04, J5 CONN_02X05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

Commit message: working on Agro_Doctor
Changed lines of the file:
@@
 Wire Wire Line
 	8150 5375 7900 5375
+Text Label 8550 6700 0    60   ~ 0
+encoder
+Text Label 8550 6800 0    60   ~ 0
+linetracker
+Text Label 8550 6900 0    60   ~ 0
+u-usb
 $EndSCHEMATC
