File: Agro_Doctor/Agro_doctor.sch (KiCad schematic (older format))
At the start: 49 parts, among them J1 Bluetooth, J10 M2, J11 M3, J12 Power_Motor, J13 MS_Conn, J2 Bluetooth, J3 3STEPPER,1SERVO, J4 Bluetooth, J5 Encoders, Stepper1, J6 3 MPU, HUMIDITY, PH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

Commit message: added the minor project file
Parts:
- removed C12, C2: 10uf, modFiles:Capacitor_10uF, symbol C
- added C10, C12, C13, C2, C3, C4, C5, C6, C7, C8, C9: C, modFiles:Capacitor_Disc_Small, symbol Device:C
- added J14, J15, J16: Conn_01x01, Pin_Headers:Pin_Header_Straight_1x01_Pitch2.54mm, symbol conn:Conn_01x01
- added J17: Conn_01x01, Pin_Headers:Pin_Header_Angled_1x01_Pitch2.54mm, symbol conn:Conn_01x01
- added J18: GND_5V, Pin_Headers:Pin_Header_Straight_2x03_Pitch2.54mm, symbol conn:Conn_02x03_Odd_Even
- added JP1, JP2, JP3, JP4, JP5, JP6: Jumper, modFiles:Resistor_small, symbol Device:Jumper
- C1, C11: symbol C -> Device:C
- D1, D3, D4: symbol LED -> Device:LED
- D2, D5: symbol D -> Device:D
- F1, F2, F3: symbol Fuse -> Device:Fuse
- J1: value Bluetooth -> Bluetooth_1; footprint Pin_Headers:Pin_Header_Straight_1x06_Pitch2.54mm -> modFiles:Bluetooth_horizontal; symbol Conn_01x06 -> conn:Conn_01x06
- J10, J11, J12, J7, J8, J9: symbol Conn_01x02 -> conn:Conn_01x02
- J13: symbol Conn_02x03_Counter_Clockwise -> conn:Conn_02x03_Counter_Clockwise
- J2: value Bluetooth -> Bluetooth_2; footprint Pin_Headers:Pin_Header_Straight_1x06_Pitch2.54mm -> modFiles:Bluetooth_horizontal; symbol Conn_01x06 -> conn:Conn_01x06
- J3, J5: symbol DB15_Female_MountingHoles -> conn:DB15_Female_MountingHoles
- J4: value Bluetooth -> Bluetooth_3; footprint Pin_Headers:Pin_Header_Straight_1x06_Pitch2.54mm -> modFiles:Bluetooth_horizontal; symbol Conn_01x06 -> conn:Conn_01x06
- J6: symbol DB9_Female_MountingHoles -> conn:DB9_Female_MountingHoles
- R1, R10, R11, R13, R2, R3, R4, R5, R6, R7, R8, R9: symbol R -> Device:R
- R12: value R -> 1k5; symbol R -> Device:R
- SW1: value SW_DIP_x01 -> Power; symbol SW_DIP_x01 -> switches:SW_DIP_x01
- U1: symbol Motor_Driver -> Prashant_library:Motor_Driver
- U10, U8: symbol Buck -> Prashant_library:Buck
- U2, U3, U4, U5: symbol A4988 -> Prashant_library:A4988
- U6, U7: symbol L298 -> Prashant_library:L298
- U9: symbol STM32F407_Discovery -> Prashant_library:STM32F407_Discovery
Connections:
- net labels added: M1_PWM, S1_DIR, S1_STEP, S2_DIR, S2_STEP, S3_DIR, S3_STEP, S4_DIR, S4_STEP
- wire segments 69 -> 119
Other:
- moved on the sheet: J10, J11, J6, J8, J9, U2, U3, U4, U5
