File: Automatic3.0/button_switches/button_switches.sch (KiCad schematic (older format))
At the start: 37 parts, among them J1 DB9_Female_MountingHoles, J2 Conn_01x01, J3 Conn_01x01, J4 Conn_01x01, J5 Conn_01x01, SW1 SW_DPST, SW2 SW_DPST, SW3 SW_DPST, SW4 SW_DPST, SW5 SW_DPST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

Commit message: added the minor project file
Parts:
- C1, C2, C3, C4, C5, C6: symbol C -> Device:C
- D1, D2, D3, D4, D5, D6, D7: symbol LED -> Device:LED
- J1: symbol DB9_Female_MountingHoles -> conn:DB9_Female_MountingHoles
- J2, J3, J4, J5: symbol Conn_01x01 -> conn:Conn_01x01
- R1, R10, R11, R12, R13, R14, R2, R3, R4, R5, R6, R7, R9: symbol R -> Device:R
- SW1, SW2, SW3, SW4, SW5, SW6: symbol SW_DPST -> switches:SW_DPST
Connections:
- wire segments 29 -> 65
