File: ir/ir.sch (KiCad schematic (older format))
At the start: 11 parts, among them P1 CONN_2, P2 CONN_1, U1 LM7809CT, U2 LM741

Commit message: added the minor project file
Parts:
- C1, C2: symbol C -> ir-rescue:C
- D1, D2: symbol LED -> ir-rescue:LED
- P1: symbol CONN_2 -> ir-rescue:CONN_2
- P2: symbol CONN_1 -> ir-rescue:CONN_1
- R1, R2: symbol R -> ir-rescue:R
- RV1: symbol POT -> ir-rescue:POT
- U1: symbol LM7809CT -> ir-rescue:LM7809CT
- U2: symbol LM741 -> ir-rescue:LM741
Changed lines of the file:
@@
-EESchema Schematic File Version 2
-LIBS:power
-LIBS:device
-LIBS:transistors
-LIBS:conn
-LIBS:linear
-LIBS:regul
-LIBS:74xx
-LIBS:cmos4000
-LIBS:adc-dac
-LIBS:memory
-LIBS:xilinx
-LIBS:special
-LIBS:microcontrollers
-LIBS:dsp
-LIBS:microchip
-LIBS:analog_switches
-LIBS:motorola
-LIBS:texas
-LIBS:intel
-LIBS:audio
-LIBS:interface
-LIBS:digital-audio
-LIBS:philips
-LIBS:display
-LIBS:cypress
-LIBS:siliconi
-LIBS:opto
-LIBS:atmel
-LIBS:contrib
-LIBS:valves
-EELAYER 25 0
+EESchema Schematic File Version 4
+LIBS:ir-cache
+EELAYER 26 0
 EELAYER END
 $Descr A4 11693 8268
@@
 $EndDescr
 $Comp
-L LM741 U2
+L ir-rescue:LM741 U2
 U 1 1 5A145632
 P 5450 3450
@@
 gnd
 $Comp
-L LM7809CT U1
+L ir-rescue:LM7809CT U1
 U 1 1 5A1456EE
 P 2850 2950
@@
 in2
 $Comp
-L POT RV1
+L ir-rescue:POT RV1
 U 1 1 5A1457A2
 P 4000 3000
@@
 vcc
 $Comp
-L R R2
+L ir-rescue:R R2
 U 1 1 5A14589D
 P 3800 3850
@@
 $EndComp
 $Comp
-L LED D2
+L ir-rescue:LED D2
 U 1 1 5A145912
 P 3800 4350
@@
 gnd
 $Comp
-L R R1
+L ir-rescue:R R1
 U 1 1 5A1459BE
 P 3100 3800
@@
 $EndComp
 $Comp
-L LED D1
+L ir-rescue:LED D1
 U 1 1 5A1459FD
 P 3100 4350
@@
 gnd
 $Comp
-L C C1
+L ir-rescue:C C1
 U 1 1 5A145C93
 P 2450 3150
@@
 $EndComp
 $Comp
-L C C2
+L ir-rescue:C C2
 U 1 1 5A145CE1
 P 3250 3150
@@
 	2450 2900 2450 2950
 Wire Wire Line
-	2450 3350 3250 3350
+	2450 3350 2850 3350
 Wire Wire Line
 	2850 3350 2850 3200
@@
 Connection ~ 2850 3350
 $Comp
-L CONN_2 P1
+L ir-rescue:CONN_2 P1
 U 1 1 5A14657F
 P 2250 2600
@@
 gnd
 $Comp
-L CONN_1 P2
+L ir-rescue:CONN_1 P2
 U 1 1 5A1467C6
 P 6450 3450
@@
 Wire Wire Line
 	6300 3450 5950 3450
+Wire Wire Line
+	2850 3350 3250 3350
 $EndSCHEMATC
