File: proximityLogic/proximityLogic.sch (KiCad schematic (older format))
At the start: 4 parts, among them J1 proximity, J2 mcu

Commit message: added the minor project file
Parts:
- D1: symbol D -> Device:D
- J1, J2: symbol Conn_01x03 -> conn:Conn_01x03
- R1: symbol R -> Device:R
Changed lines of the file:
@@
-EESchema Schematic File Version 2
-LIBS:power
-LIBS:device
-LIBS:switches
-LIBS:relays
-LIBS:motors
-LIBS:transistors
-LIBS:conn
-LIBS:linear
-LIBS:regul
-LIBS:74xx
-LIBS:cmos4000
-LIBS:adc-dac
-LIBS:memory
-LIBS:xilinx
-LIBS:microcontrollers
-LIBS:dsp
-LIBS:microchip
-LIBS:analog_switches
-LIBS:motorola
-LIBS:texas
-LIBS:intel
-LIBS:audio
-LIBS:interface
-LIBS:digital-audio
-LIBS:philips
-LIBS:display
-LIBS:cypress
-LIBS:siliconi
-LIBS:opto
-LIBS:atmel
-LIBS:contrib
-LIBS:valves
-EELAYER 25 0
+EESchema Schematic File Version 4
+LIBS:proximityLogic-cache
+EELAYER 26 0
 EELAYER END
 $Descr A4 11693 8268
@@
 $EndDescr
 $Comp
-L D D1
+L Device:D D1
 U 1 1 5B673752
 P 5350 3975
@@
 $EndComp
 $Comp
-L R R1
+L Device:R R1
 U 1 1 5B6737FA
 P 5500 3825
@@
 $EndComp
 $Comp
-L Conn_01x03 J2
+L conn:Conn_01x03 J2
 U 1 1 5B673885
 P 5900 3975
@@
 	5500 3975 5700 3975
 $Comp
-L Conn_01x03 J1
+L conn:Conn_01x03 J1
 U 1 1 5B673933
 P 5000 3975
@@
 $EndComp
 $Comp
-L +12V #PWR01
+L power:+12V #PWR01
 U 1 1 5B673A08
 P 5200 3875
@@
 $EndComp
 $Comp
-L +12V #PWR02
+L power:+12V #PWR02
 U 1 1 5B673A8C
 P 5700 3875
@@
 $EndComp
 $Comp
-L GND #PWR03
+L power:GND #PWR03
 U 1 1 5B673AA1
 P 5200 4075
@@
 $EndComp
 $Comp
-L GND #PWR04
+L power:GND #PWR04
 U 1 1 5B673ABF
 P 5700 4075
@@
 $EndComp
 $Comp
-L +12V #PWR05
+L power:+12V #PWR05
 U 1 1 5B673B0A
 P 5500 3675
